File: Hardware/Production/Artemis-MicroMod-Panel.brd (EAGLE design)
At the start: 199.6 x 83.1 mm, 550 parts, among them J1 MICROMOD-2222, J10 MICROMOD-2222, J11 MICROMOD-2222, J12 MICROMOD-2222, J13 MICROMOD-2222, J14 MICROMOD-2222, J15 MICROMOD-2222, J16 MICROMOD-2222, J2 MICROMOD-2222, J3 MICROMOD-2222, J4 MICROMOD-2222, J5 MICROMOD-2222, J6 MICROMOD-2222, J7 MICROMOD-2222, J8 MICROMOD-2222, J9 MICROMOD-2222, U1 ARTEMIS_MODULESMD, U10 ARTEMIS_MODULESMD, U11 CH340E_MSOP10, U12 TSV524, U13 ARTEMIS_MODULESMD, U14 CH340E_MSOP10, U15 TSV524, U16 ARTEMIS_MODULESMD, U17 CH340E_MSOP10, U18 TSV524, U19 ARTEMIS_MODULESMD, U2 TSV524, U20 CH340E_MSOP10, U21 TSV524, U22 ARTEMIS_MODULESMD, U23 CH340E_MSOP10, U24 TSV524, U25 ARTEMIS_MODULESMD, U26 CH340E_MSOP10, U27 TSV524, U28 ARTEMIS_MODULESMD, U29 CH340E_MSOP10, U3 ARTEMIS_MODULESMD, U30 TSV524, U31 ARTEMIS_MODULESMD, U32 CH340E_MSOP10, U33 TSV524, U34 ARTEMIS_MODULESMD, U35 CH340E_MSOP10, U36 TSV524, U37 ARTEMIS_MODULESMD, U38 CH340E_MSOP10, U39 TSV524, U4 CH340E_MSOP10, U40 ARTEMIS_MODULESMD, U41 CH340E_MSOP10, U42 TSV524, U43 ARTEMIS_MODULESMD, U44 CH340E_MSOP10, U45 TSV524, U46 ARTEMIS_MODULESMD, U47 CH340E_MSOP10, U48 TSV524, U5 TSV524, U6 CH340E_MSOP10, U7 ARTEMIS_MODULESMD, U8 CH340E_MSOP10, U9 TSV524, Y1 32.768kHz, Y10 32.768kHz, Y11 32.768kHz, Y12 32.768kHz, Y13 32.768kHz, Y14 32.768kHz, Y15 32.768kHz, Y16 32.768kHz, Y2 32.768kHz, Y3 32.768kHz, Y4 32.768kHz, Y5 32.768kHz, Y6 32.768kHz, Y7 32.768kHz, Y8 32.768kHz, Y9 32.768kHz

Commit message: Add v1.1 production files
Parts:
- moved R133 2.01 mm to (145.0, 64.9), turned to 180 degrees
- moved R142 2.01 mm to (167.5, 64.9), turned to 180 degrees
- moved R61 2.01 mm to (147.1, 4.95), turned to 0 degrees
- moved R70 2.01 mm to (169.6, 4.95), turned to 0 degrees
- moved R34 2.01 mm to (79.5, 4.95), turned to 0 degrees
- moved R97 2.01 mm to (55.0, 64.9), turned to 180 degrees
- moved R5 2.01 mm to (12.0, 4.95), turned to 0 degrees
- moved R79 2.01 mm to (9.99, 64.9), turned to 180 degrees
- moved R16 2.01 mm to (34.5, 4.95), turned to 0 degrees
- moved R25 2.01 mm to (57.0, 4.95), turned to 0 degrees
- moved R88 2.01 mm to (32.5, 64.9), turned to 180 degrees
- moved R106 2.01 mm to (77.5, 64.9), turned to 180 degrees
- moved R115 2.01 mm to (100.0, 64.9), turned to 180 degrees
- moved R124 2.01 mm to (122.5, 64.9), turned to 180 degrees
- moved R43 2.01 mm to (102.0, 4.95), turned to 0 degrees
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Connections:
- net N$103 renamed ADC1_BUFF15
- net N$104 renamed ADC0_BUFF29
- net N$110 renamed ADC1_BUFF16
- net N$111 renamed ADC0_BUFF31
- net N$12 renamed ADC1_BUFF1
- net N$13 renamed ADC0_BUFF3
- net N$19 renamed ADC1_BUFF3
- net N$20 renamed ADC0_BUFF5
- net N$26 renamed ADC1_BUFF4
- net N$27 renamed ADC0_BUFF7
- net N$3 renamed ADC1_BUFF2
- net N$33 renamed ADC1_BUFF5
- net N$34 renamed ADC0_BUFF9
- net N$40 renamed ADC1_BUFF6
- net N$41 renamed ADC0_BUFF11
- net N$47 renamed ADC1_BUFF7
- net N$48 renamed ADC0_BUFF13
- net N$54 renamed ADC1_BUFF8
- net N$55 renamed ADC0_BUFF15
- net N$61 renamed ADC1_BUFF9
- net N$62 renamed ADC0_BUFF17
- net N$68 renamed ADC1_BUFF10
- net N$69 renamed ADC0_BUFF19
- net N$75 renamed ADC1_BUFF11
- net N$76 renamed ADC0_BUFF21
- net N$82 renamed ADC1_BUFF12
- net N$83 renamed ADC0_BUFF23
- net N$89 renamed ADC1_BUFF13
- net N$9 renamed ADC0_BUFF2
- net N$90 renamed ADC0_BUFF25
- net N$96 renamed ADC1_BUFF14
- net N$97 renamed ADC0_BUFF27
- removed net N$10 (its old number): R2.1, R4.2, U2.1
- removed net N$105: R130.1, R131.2, U45.1
- removed net N$112: R139.1, R140.2, U48.1
- removed net N$14 (its old number): R11.1, R12.2, U5.1
- removed net N$21 (its old number): R22.1, R23.2, U9.1
- removed net N$28 (its old number): R31.1, R32.2, U12.1
- removed net N$35 (its old number): R40.1, R41.2, U15.1
- removed net N$42 (its old number): R49.1, R50.2, U18.1
- removed net N$49 (its old number): R58.1, R59.2, U21.1
- removed net N$56 (its old number): R67.1, R68.2, U24.1
- removed net N$63 (its old number): R76.1, R77.2, U27.1
- removed net N$70: R85.1, R86.2, U30.1
- removed net N$77: R94.1, R95.2, U33.1
- removed net N$84: R103.1, R104.2, U36.1
- removed net N$91: R112.1, R113.2, U39.1
- removed net N$98: R121.1, R122.2, U42.1
- new net ADC0_BUFF1: R3.2, U2.15, U2.16
- new net ADC0_BUFF10: R42.2, U15.15, U15.16
- new net ADC0_BUFF12: R51.2, U18.15, U18.16
- new net ADC0_BUFF14: R60.2, U21.15, U21.16
- new net ADC0_BUFF16: R69.2, U24.15, U24.16
- new net ADC0_BUFF18: R78.2, U27.15, U27.16
- new net ADC0_BUFF20: R87.2, U30.15, U30.16
- new net ADC0_BUFF22: R96.2, U33.15, U33.16
- new net ADC0_BUFF24: R105.2, U36.15, U36.16
- new net ADC0_BUFF26: R114.2, U39.15, U39.16
- new net ADC0_BUFF28: R123.2, U42.15, U42.16
- new net ADC0_BUFF30: R132.2, U45.15, U45.16
- new net ADC0_BUFF32: R141.2, U48.15, U48.16
- new net ADC0_BUFF4: R13.2, U5.15, U5.16
- new net ADC0_BUFF6: R24.2, U9.15, U9.16
- new net ADC0_BUFF8: R33.2, U12.15, U12.16
- new net ADC_BUFF1: R6.2, U2.13, U2.14
- new net ADC_BUFF10: R89.2, U30.13, U30.14
- new net ADC_BUFF11: R98.2, U33.13, U33.14
- new net ADC_BUFF12: R107.2, U36.13, U36.14
- new net ADC_BUFF13: R116.2, U39.13, U39.14
- new net ADC_BUFF14: R125.2, U42.13, U42.14
- new net ADC_BUFF15: R134.2, U45.13, U45.14
- new net ADC_BUFF16: R143.2, U48.13, U48.14
- new net ADC_BUFF2: R17.2, U5.13, U5.14
- new net ADC_BUFF3: R26.2, U9.13, U9.14
- new net ADC_BUFF4: R35.2, U12.13, U12.14
- new net ADC_BUFF5: R44.2, U15.13, U15.14
- new net ADC_BUFF6: R53.2, U18.13, U18.14
- new net ADC_BUFF7: R62.2, U21.13, U21.14
- new net ADC_BUFF8: R71.2, U24.13, U24.14
- new net ADC_BUFF9: R80.2, U27.13, U27.14
- net ADC0: now also U2.1; no longer R3.2
- net ADC1: now also U2.12; no longer R6.2
- net ADC10: now also U18.1; no longer R51.2
- net ADC11: now also U18.12; no longer R53.2
- net ADC12: now also U21.1; no longer R60.2
- net ADC13: now also U21.12; no longer R62.2
- net ADC14: now also U24.1; no longer R69.2
- net ADC15: now also U24.12; no longer R71.2
- net ADC16: now also U27.1; no longer R78.2
- net ADC17: now also U27.12; no longer R80.2
- net ADC18: now also U30.1; no longer R87.2
- net ADC19: now also U30.12; no longer R89.2
- net ADC2: now also U5.1; no longer R13.2
- net ADC20: now also U33.1; no longer R96.2
- net ADC21: now also U33.12; no longer R98.2
- net ADC22: now also U36.1; no longer R105.2
- net ADC23: now also U36.12; no longer R107.2
- net ADC24: now also U39.1; no longer R114.2
- net ADC25: now also U39.12; no longer R116.2
- net ADC26: now also U42.1; no longer R123.2
- net ADC27: now also U42.12; no longer R125.2
- net ADC28: now also U45.1; no longer R132.2
- net ADC29: now also U45.12; no longer R134.2
- net ADC3: now also U5.12; no longer R17.2
- net ADC30: now also U48.1; no longer R141.2
- net ADC31: now also U48.12; no longer R143.2
- net ADC4: now also U9.1; no longer R24.2
- net ADC5: now also U9.12; no longer R26.2
- net ADC6: now also U12.1; no longer R33.2
- net ADC7: now also U12.12; no longer R35.2
- net ADC8: now also U15.1; no longer R42.2
- net ADC9: now also U15.12; no longer R44.2
- net SCALED_BATT_VIN/1: now also R11.1, R12.2; no longer U5.15, U5.16
- net SCALED_BATT_VIN/10: now also R85.1, R86.2; no longer U30.15, U30.16
- net SCALED_BATT_VIN/11: now also R94.1, R95.2; no longer U33.15, U33.16
- net SCALED_BATT_VIN/12: now also R103.1, R104.2; no longer U36.15, U36.16
- net SCALED_BATT_VIN/13: now also R112.1, R113.2; no longer U39.15, U39.16
- net SCALED_BATT_VIN/14: now also R121.1, R122.2; no longer U42.15, U42.16
- net SCALED_BATT_VIN/15: now also R130.1, R131.2; no longer U45.15, U45.16
- net SCALED_BATT_VIN/16: now also R139.1, R140.2; no longer U48.15, U48.16
- net SCALED_BATT_VIN/2: now also R22.1, R23.2; no longer U9.15, U9.16
- net SCALED_BATT_VIN/3: now also R2.1, R4.2; no longer U2.15, U2.16
- net SCALED_BATT_VIN/4: now also R31.1, R32.2; no longer U12.15, U12.16
- net SCALED_BATT_VIN/5: now also R40.1, R41.2; no longer U15.15, U15.16
- net SCALED_BATT_VIN/6: now also R49.1, R50.2; no longer U18.15, U18.16
- net SCALED_BATT_VIN/7: now also R58.1, R59.2; no longer U21.15, U21.16
- net SCALED_BATT_VIN/8: now also R67.1, R68.2; no longer U24.15, U24.16
- net SCALED_BATT_VIN/9: now also R76.1, R77.2; no longer U27.15, U27.16
Routing:
- net ADC0_BUFF26: track 0.00 -> 5.67 mm
- net ADC0_BUFF20: track 0.00 -> 5.67 mm
- net ADC0_BUFF10: track 0.00 -> 5.67 mm
- net ADC0_BUFF18: track 0.00 -> 5.67 mm
- net ADC0_BUFF22: track 0.00 -> 5.67 mm
- net ADC0_BUFF28: track 0.00 -> 5.67 mm
- net ADC0_BUFF24: track 0.00 -> 5.67 mm
- net ADC0_BUFF1: track 0.00 -> 5.67 mm
- net ADC0_BUFF8: track 0.00 -> 5.67 mm
- net ADC0_BUFF6: track 0.00 -> 5.67 mm
- net ADC0_BUFF4: track 0.00 -> 5.67 mm
- net ADC0_BUFF32: track 0.00 -> 5.67 mm
- net ADC0_BUFF30: track 0.00 -> 5.67 mm
- net ADC0_BUFF12: track 0.00 -> 5.67 mm
- net ADC0_BUFF16: track 0.00 -> 5.67 mm
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
Commit message: Route from opamp for better AOI. fix DRC error. Add v1.2 panel files.
Parts:
- added C129, C130, C137, C138, C145, C146, C153, C154: 15pF, SparkFun-Capacitors:0402-TIGHT
- added C131, C139, C147, C155: 10nF, SparkFun-Capacitors:0402-TIGHT
- added C132, C133, C134, C136, C140, C141, C142, C144, C148, C149, C150, C152, C156, C157, C158, C160: 0.1uF, SparkFun-Capacitors:0402-TIGHT
- added C135, C143, C151, C159: 1.0nF, SparkFun-Capacitors:0402-TIGHT
- added D17, D19, D21, D23, D25, D27, D29, D31, D33, D35, D37, D39: BLUE, SparkFun-LED:LED-0603
- added D18, D20, D22, D24, D26, D28, D30, D32, D34, D36, D38, D40: 1A/23V/620mV, SparkFun-DiscreteSemi:SOD-323
- added FD65, FD66, FD67, FD68, FD69, FD70, FD71, FD72, FD73, FD74, FD75, FD76, FD77, FD78, FD79, FD80: FIDUCIALUFIDUCIAL, SparkFun-Aesthetics:FIDUCIAL-MICRO
- added J17, J18, J19, J20: MICROMOD-2222, SparkFun-MicroMod:M.2-CARD-E-22
- added LOGO33, LOGO36, LOGO39, LOGO42, LOGO45, LOGO48, LOGO51, LOGO54, LOGO57, LOGO60: SFE_LOGO_FLAME.1_INCH, SparkFun-Aesthetics:SFE_LOGO_FLAME_.1
- added LOGO34, LOGO37, LOGO40, LOGO43, LOGO46, LOGO49, LOGO52, LOGO55, LOGO58: OSHW-LOGOMINI, SparkFun-Aesthetics:OSHW-LOGO-MINI
- added LOGO35, LOGO38, LOGO41, LOGO44, LOGO47, LOGO50, LOGO53, LOGO56, LOGO59: SFE_LOGO_NAME_FLAME.1_INCH, SparkFun-Aesthetics:SFE_LOGO_NAME_FLAME_.1
- added R145, R154, R163, R172: 1k, SparkFun-Resistors:0402-TIGHT
- added R146, R148, R150, R152, R155, R157, R159, R161, R164, R166, R168, R170, R173, R175, R177, R179: 100k, SparkFun-Resistors:0402-TIGHT
- added R147, R156, R165, R174: 220KOHM-0402T-1/16W-1%, SparkFun-Resistors:0402-TIGHT
- added R149, R151, R153, R158, R160, R162, R167, R169, R171, R176, R178, R180: 150k, SparkFun-Resistors:0402-TIGHT
- added U$100, U$107, U$114, U$121, U$128, U$135, U$86, U$93: (no value), buzzard_labels:MICROMOD1
- added U$101, U$108, U$115, U$122, U$129, U$136, U$87, U$94: (no value), buzzard_labels (1):ARTEMIS2
- added U$102, U$109, U$116, U$123, U$130, U$137, U$81, U$88, U$95: (no value), SparkFun-Buzzard:STAT_TO_32
- added U$103, U$105, U$110, U$112, U$117, U$119, U$124, U$126, U$131, U$133, U$138, U$140, U$82, U$84, U$89, U$91, U$96, U$98: (no value), SparkFun-MicroMod:MICROMOD_MI_LOGO_.35
- added U$104, U$111, U$118, U$125, U$132, U$139, U$83, U$90, U$97: (no value), SparkFun-MicroMod:MICROMOD_LOGO_.35
- added U$106, U$113, U$120, U$127, U$134, U$85, U$92, U$99: (no value), buzzard_labels:ARTEMIS0
- added U49, U52, U55, U58: ARTEMIS_MODULESMD, SparkFun-IC-Microcontroller:ARTEMIS_FP
- added U50, U53, U56, U59: CH340E_MSOP10, SparkFun-IC-Comms:MSOP10
- added U51, U54, U57, U60: TSV524, OpAmp:QFN-16
- added Y17, Y18, Y19, Y20: 32.768kHz, SparkFun-Clocks:CRYSTAL-SMD-3.2X1.5MM
- D10, D12, D14, D16, D3, D5, D7, D8: value BLUE -> 1A/23V/620mV; device SparkFun-LED:LED-0603 -> SparkFun-DiscreteSemi:SOD-323
- LOGO10, LOGO16, LOGO22, LOGO28, LOGO4: value SFE_LOGO_NAME_FLAME.1_INCH -> OSHW-LOGOMINI; device SparkFun-Aesthetics:SFE_LOGO_NAME_FLAME_.1 -> SparkFun-Aesthetics:OSHW-LOGO-MINI
- LOGO11, LOGO17, LOGO23, LOGO29, LOGO5: value OSHW-LOGOMINI -> SFE_LOGO_NAME_FLAME.1_INCH; device SparkFun-Aesthetics:OSHW-LOGO-MINI -> SparkFun-Aesthetics:SFE_LOGO_NAME_FLAME_.1
- LOGO12, LOGO18, LOGO24, LOGO30, LOGO6: value SFE_LOGO_NAME_FLAME.1_INCH -> SFE_LOGO_FLAME.1_INCH; device SparkFun-Aesthetics:SFE_LOGO_NAME_FLAME_.1 -> SparkFun-Aesthetics:SFE_LOGO_FLAME_.1
- LOGO15, LOGO2, LOGO21, LOGO27, LOGO9: value OSHW-LOGOMINI -> SFE_LOGO_FLAME.1_INCH; device SparkFun-Aesthetics:OSHW-LOGO-MINI -> SparkFun-Aesthetics:SFE_LOGO_FLAME_.1
- U$1, U$21, U$26, U$56, U$61: device SparkFun-Buzzard:STAT_32 -> SparkFun-MicroMod:MICROMOD_MI_LOGO_.35
- U$10, U$45, U$80: device buzzard_labels (1):MICROMOD1 -> buzzard_labels (1):ARTEMIS2
- U$11, U$4, U$46: device SparkFun-Buzzard:STAT_32 -> SparkFun-Buzzard:STAT_TO_32
- U$12, U$42, U$47, U$77: device buzzard_labels:ARTEMIS0 -> SparkFun-MicroMod:MICROMOD_MI_LOGO_.35
- U$13, U$48: device buzzard_labels:MICROMOD1 -> SparkFun-MicroMod:MICROMOD_LOGO_.35
- U$14, U$19, U$49, U$54: device buzzard_labels (1):ARTEMIS2 -> SparkFun-MicroMod:MICROMOD_MI_LOGO_.35
- U$15, U$50: device buzzard_labels (1):MICROMOD1 -> buzzard_labels:ARTEMIS0
- U$16, U$51: device SparkFun-Buzzard:STAT_32 -> buzzard_labels:MICROMOD1
- U$17, U$52: device buzzard_labels:ARTEMIS0 -> buzzard_labels (1):ARTEMIS2
- U$18, U$53: device buzzard_labels:MICROMOD1 -> SparkFun-Buzzard:STAT_TO_32
- U$20, U$55: device buzzard_labels (1):MICROMOD1 -> SparkFun-MicroMod:MICROMOD_LOGO_.35
- U$25, U$60: device buzzard_labels (1):MICROMOD1 -> SparkFun-Buzzard:STAT_TO_32
- U$27, U$5, U$62: device buzzard_labels:ARTEMIS0 -> SparkFun-MicroMod:MICROMOD_LOGO_.35
- U$28, U$33, U$63, U$68: device buzzard_labels:MICROMOD1 -> SparkFun-MicroMod:MICROMOD_MI_LOGO_.35
- U$29, U$64: device buzzard_labels (1):ARTEMIS2 -> buzzard_labels:ARTEMIS0
- U$30, U$65: device buzzard_labels (1):MICROMOD1 -> buzzard_labels:MICROMOD1
- U$31, U$66: device SparkFun-Buzzard:STAT_32 -> buzzard_labels (1):ARTEMIS2
- U$32, U$67: device buzzard_labels:ARTEMIS0 -> SparkFun-Buzzard:STAT_TO_32
- U$34, U$69: device buzzard_labels (1):ARTEMIS2 -> SparkFun-MicroMod:MICROMOD_LOGO_.35
- U$35, U$40, U$7, U$70, U$75: device buzzard_labels (1):MICROMOD1 -> SparkFun-MicroMod:MICROMOD_MI_LOGO_.35
- U$36, U$71: device SparkFun-Buzzard:STAT_32 -> buzzard_labels:ARTEMIS0
- U$37, U$72: device buzzard_labels:ARTEMIS0 -> buzzard_labels:MICROMOD1
- U$38, U$73: device buzzard_labels:MICROMOD1 -> buzzard_labels (1):ARTEMIS2
- U$39, U$74: device buzzard_labels (1):ARTEMIS2 -> SparkFun-Buzzard:STAT_TO_32
- U$41, U$76: device SparkFun-Buzzard:STAT_32 -> SparkFun-MicroMod:MICROMOD_LOGO_.35
- U$43, U$78, U$8: device buzzard_labels:MICROMOD1 -> buzzard_labels:ARTEMIS0
- U$44, U$79, U$9: device buzzard_labels (1):ARTEMIS2 -> buzzard_labels:MICROMOD1
- moved C67 205.3 mm to (201.1, 12.0), turned to 270 degrees
- moved C75 205.3 mm to (223.6, 12.0), turned to 270 degrees
- moved C65 204.2 mm to (200.3, 11.0), turned to 90 degrees
- moved C73 204.2 mm to (222.8, 11.0), turned to 90 degrees
- moved Y10 202.8 mm to (222.8, 14.0), turned to 270 degrees
- moved Y9 202.8 mm to (200.3, 14.0), turned to 270 degrees
- moved FD34 202.2 mm to (201.4, 21.3), turned to 0 degrees
- moved FD38 202.2 mm to (223.9, 21.3), turned to 0 degrees
- moved FD35 202.0 mm to (201.1, 21.0), turned to 0 degrees
- moved FD39 202.0 mm to (223.6, 21.0), turned to 0 degrees
- moved C66 201.7 mm to (200.3, 17.0), turned to 270 degrees
- moved C74 201.7 mm to (222.8, 17.0), turned to 270 degrees
- moved U26 199.4 mm to (198.1, 12.0), turned to 90 degrees
- moved U29 199.4 mm to (220.6, 12.0), turned to 90 degrees
- moved C68 193.6 mm to (195.1, 12.0), turned to 270 degrees
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Connections:
- net SDIO_DATA41 renamed SPI_!CS!20
- net SDIO_DATA44 renamed SPI_MISO22
- net SDIO_DATA45 renamed SPI_!CS!22
- net SDIO_DATA48 renamed SPI_MISO24
- net SDIO_DATA49 renamed SPI_!CS!24
- net SDIO_DATA52 renamed SPI_MISO26
- net SDIO_DATA53 renamed SPI_!CS!26
- net SDIO_DATA56 renamed SPI_MISO28
- net SDIO_DATA57 renamed SPI_!CS!28
- net SDIO_DATA60 renamed SPI_MISO30
- net SDIO_DATA61 renamed SPI_!CS!30
- removed net SDIO_DATA0: J1.64, U1.~D22, U1.~D6
- removed net SDIO_DATA42: J11.66, U31.~D26
- removed net SDIO_DATA43: J11.68, U31.~D4
- removed net SDIO_DATA46: J12.66, U34.~D26
- removed net SDIO_DATA47: J12.68, U34.~D4
- removed net SDIO_DATA50: J13.66, U37.~D26
- removed net SDIO_DATA51: J13.68, U37.~D4
- removed net SDIO_DATA54: J14.66, U40.~D26
- removed net SDIO_DATA55: J14.68, U40.~D4
- removed net SDIO_DATA58: J15.66, U43.~D26
- removed net SDIO_DATA59: J15.68, U43.~D4
- removed net SDIO_DATA62: J16.66, U46.~D26
- removed net SDIO_DATA63: J16.68, U46.~D4
- new net !RESET!16: C133.2, C135.1, J17.6, R146.1, U49.~RST
- new net !RESET!17: C141.2, C143.1, J18.6, R155.1, U52.~RST
- new net !RESET!18: C149.2, C151.1, J19.6, R164.1, U55.~RST
- new net !RESET!19: C157.2, C159.1, J20.6, R173.1, U58.~RST
- new net !RTS16: C133.1, C134.1, U50.4
- new net !RTS17: C141.1, C142.1, U53.4
- new net !RTS18: C149.1, C150.1, U56.4
- new net !RTS19: C157.1, C158.1, U59.4
- new net 3.3V16: C131.1, C132.1, C136.1, D34.C, J17.72, R146.2, U49.VDD@36, U49.VDD@37, U50.10, U50.7, U51.2
- new net 3.3V17: C139.1, C140.1, C144.1, D36.C, J18.72, R155.2, U52.VDD@36, U52.VDD@37, U53.10, U53.7, U54.2
- new net 3.3V18: C147.1, C148.1, C152.1, D38.C, J19.72, R164.2, U55.VDD@36, U55.VDD@37, U56.10, U56.7, U57.2
- new net 3.3V19: C155.1, C156.1, C160.1, D40.C, J20.72, R173.2, U58.VDD@36, U58.VDD@37, U59.10, U59.7, U60.2
- new net 3.3V_EN16: J17.4, U49.D3
- new net 3.3V_EN17: J18.4, U52.D3
- new net 3.3V_EN18: J19.4, U55.D3
- new net 3.3V_EN19: J20.4, U58.D3
- new net 3.3V_MAIN: D7.A, J1.2, J1.74
- new net 3.3V_MAIN1: D3.A, J2.2, J2.74
- new net 3.3V_MAIN10: D22.A, J11.2, J11.74
- new net 3.3V_MAIN11: D24.A, J12.2, J12.74
- new net 3.3V_MAIN12: D26.A, J13.2, J13.74
- new net 3.3V_MAIN13: D28.A, J14.2, J14.74
- new net 3.3V_MAIN14: D30.A, J15.2, J15.74
- new net 3.3V_MAIN15: D32.A, J16.2, J16.74
- new net 3.3V_MAIN16: D34.A, J17.2, J17.74
- new net 3.3V_MAIN17: D36.A, J18.2, J18.74
- new net 3.3V_MAIN18: D38.A, J19.2, J19.74
- new net 3.3V_MAIN19: D40.A, J20.2, J20.74
- new net 3.3V_MAIN2: D5.A, J3.2, J3.74
- new net 3.3V_MAIN3: D8.A, J4.2, J4.74
- new net 3.3V_MAIN4: D10.A, J5.2, J5.74
- new net 3.3V_MAIN5: D12.A, J6.2, J6.74
- new net 3.3V_MAIN6: D14.A, J7.2, J7.74
- new net 3.3V_MAIN7: D16.A, J8.2, J8.74
- new net 3.3V_MAIN8: D18.A, J9.2, J9.74
- new net 3.3V_MAIN9: D20.A, J10.2, J10.74
- new net ADC0_BUFF33: R150.1, R151.2, U51.4
- new net ADC0_BUFF34: R150.2, U51.15, U51.16
- new net ADC0_BUFF35: R159.1, R160.2, U54.4
- new net ADC0_BUFF36: R159.2, U54.15, U54.16
- new net ADC0_BUFF37: R168.1, R169.2, U57.4
- new net ADC0_BUFF38: R168.2, U57.15, U57.16
- new net ADC0_BUFF39: R177.1, R178.2, U60.4
- new net ADC0_BUFF40: R177.2, U60.15, U60.16
- new net ADC1_BUFF17: R152.1, R153.2, U51.9
- new net ADC1_BUFF18: R161.1, R162.2, U54.9
- new net ADC1_BUFF19: R170.1, R171.2, U57.9
- new net ADC1_BUFF20: R179.1, R180.2, U60.9
- new net ADC32: J17.34, U51.1
- new net ADC33: J17.38, U51.12
- new net ADC34: J18.34, U54.1
- new net ADC35: J18.38, U54.12
- new net ADC36: J19.34, U57.1
- new net ADC37: J19.38, U57.12
- new net ADC38: J20.34, U60.1
- new net ADC39: J20.38, U60.12
- new net ADC_BUFF17: R152.2, U51.13, U51.14
- new net ADC_BUFF18: R161.2, U54.13, U54.14
- new net ADC_BUFF19: R170.2, U57.13, U57.14
- new net ADC_BUFF20: R179.2, U60.13, U60.14
- new net ADC_D+16: J17.63, U49.~AD13
- new net ADC_D+17: J18.63, U52.~AD13
- new net ADC_D+18: J19.63, U55.~AD13
- new net ADC_D+19: J20.63, U58.~AD13
- new net ADC_D-16: J17.65, U49.~AD12
- new net ADC_D-17: J18.65, U52.~AD12
- new net ADC_D-18: J19.65, U55.~AD12
- new net ADC_D-19: J20.65, U58.~AD12
- new net BATT_VIN/17: J17.51, R148.2
- new net BATT_VIN/18: J18.51, R157.2
- new net BATT_VIN/19: J19.51, R166.2
- new net BATT_VIN/20: J20.51, R175.2
- new net BOOT16: C134.2, J17.11, R147.2, U49.BOOT
- new net BOOT17: C142.2, J18.11, R156.2, U52.BOOT
- new net BOOT18: C150.2, J19.11, R165.2, U55.BOOT
- new net BOOT19: C158.2, J20.11, R174.2, U58.BOOT
- new net CAM_PCLK16: J17.54, U49.~AD11
- new net CAM_PCLK17: J18.54, U52.~AD11
- new net CAM_PCLK18: J19.54, U55.~AD11
- new net CAM_PCLK19: J20.54, U58.~AD11
- new net CLKOUT16: J17.56, J17.58, U49.D0
- new net CLKOUT17: J18.56, J18.58, U52.D0
- new net CLKOUT18: J19.56, J19.58, U55.D0
- new net CLKOUT19: J20.56, J20.58, U58.D0
- new net CTS17: J17.15, U49.D17
- new net CTS18: J18.15, U52.D17
- new net CTS19: J19.15, U55.D17
- new net CTS20: J20.15, U58.D17
- new net D32: J17.10, U49.D1
- new net D33: J17.18, U49.D2
- new net D34: J18.10, U52.D1
- new net D35: J18.18, U52.D2
- new net D36: J19.10, U55.D1
- new net D37: J19.18, U55.D2
- new net D38: J20.10, U58.D1
- new net D39: J20.18, U58.D2
- new net GND16: C129.1, C130.1, C131.2, C132.2, C135.2, C136.2, D33.C, J17.1, J17.33, J17.36, J17.39, J17.45, J17.7, J17.75, J17.GND1, J17.GND2, J17.GND3, R147.1, R149.1, R151.1, R153.1, U49.GND@1, U49.GND@22, U49.GND@38, U49.GND@39, U49.GND@47, U49.GND@59, U50.3, U51.11
- new net GND17: C137.1, C138.1, C139.2, C140.2, C143.2, C144.2, D35.C, J18.1, J18.33, J18.36, J18.39, J18.45, J18.7, J18.75, J18.GND1, J18.GND2, J18.GND3, R156.1, R158.1, R160.1, R162.1, U52.GND@1, U52.GND@22, U52.GND@38, U52.GND@39, U52.GND@47, U52.GND@59, U53.3, U54.11
- new net GND18: C145.1, C146.1, C147.2, C148.2, C151.2, C152.2, D37.C, J19.1, J19.33, J19.36, J19.39, J19.45, J19.7, J19.75, J19.GND1, J19.GND2, J19.GND3, R165.1, R167.1, R169.1, R171.1, U55.GND@1, U55.GND@22, U55.GND@38, U55.GND@39, U55.GND@47, U55.GND@59, U56.3, U57.11
- new net GND19: C153.1, C154.1, C155.2, C156.2, C159.2, C160.2, D39.C, J20.1, J20.33, J20.36, J20.39, J20.45, J20.7, J20.75, J20.GND1, J20.GND2, J20.GND3, R174.1, R176.1, R178.1, R180.1, U58.GND@1, U58.GND@22, U58.GND@38, U58.GND@39, U58.GND@47, U58.GND@59, U59.3, U60.11
- new net GPIO128: J17.73, U49.~AD29
- new net GPIO129: J17.69, U49.D15
- new net GPIO130: J17.71, U49.D14
- new net GPIO131: J17.42, U49.~AD33/SWO
- new net GPIO132: J17.46, U49.~D27
- new net GPIO133: J17.44, U49.AD34
- new net GPIO134: J17.48, U49.~D28
- new net GPIO135: J17.40, U49.AD16
- new net GPIO136: J18.73, U52.~AD29
- new net GPIO137: J18.69, U52.D15
- new net GPIO138: J18.71, U52.D14
- new net GPIO139: J18.42, U52.~AD33/SWO
- new net GPIO140: J18.46, U52.~D27
- new net GPIO141: J18.44, U52.AD34
- new net GPIO142: J18.48, U52.~D28
- new net GPIO143: J18.40, U52.AD16
- new net GPIO144: J19.73, U55.~AD29
- new net GPIO145: J19.69, U55.D15
- new net GPIO146: J19.71, U55.D14
- new net GPIO147: J19.42, U55.~AD33/SWO
- new net GPIO148: J19.46, U55.~D27
- new net GPIO149: J19.44, U55.AD34
- new net GPIO150: J19.48, U55.~D28
- new net GPIO151: J19.40, U55.AD16
- new net GPIO152: J20.73, U58.~AD29
- new net GPIO153: J20.69, U58.D15
- new net GPIO154: J20.71, U58.D14
- new net GPIO155: J20.42, U58.~AD33/SWO
- new net GPIO156: J20.46, U58.~D27
- new net GPIO157: J20.44, U58.AD34
- new net GPIO158: J20.48, U58.~D28
- new net GPIO159: J20.40, U58.AD16
- new net I2C_!INT!16: J17.16, U49.~D18
- new net I2C_!INT!17: J18.16, U52.~D18
- new net I2C_!INT!18: J19.16, U55.~D18
- new net I2C_!INT!19: J20.16, U58.~D18
- new net LED_BUILTIN16: R145.2, U49.~D19
- new net LED_BUILTIN17: R154.2, U52.~D19
- new net LED_BUILTIN18: R163.2, U55.~D19
- new net LED_BUILTIN19: R172.2, U58.~D19
- new net N$65: C129.2, U49.XO, Y17.P$2
- new net N$66: D33.A, R145.1
- new net N$67: U49.XI
- new net N$68: C130.2, Y17.P$1
- new net N$69: C137.2, U52.XO, Y18.P$2
- new net N$70: D35.A, R154.1
- new net N$71: U52.XI
- new net N$72: C138.2, Y18.P$1
- new net N$73: C145.2, U55.XO, Y19.P$2
- new net N$74: D37.A, R163.1
- new net N$75: U55.XI
- new net N$76: C146.2, Y19.P$1
- new net N$77: C153.2, U58.XO, Y20.P$2
- new net N$78: D39.A, R172.1
- new net N$79: U58.XI
- new net N$80: C154.2, Y20.P$1
- new net PDM_CLK16: J17.50, U49.~D37
- new net PDM_CLK17: J18.50, U52.~D37
- new net PDM_CLK18: J19.50, U55.~D37
- new net PDM_CLK19: J20.50, U58.~D37
- new net PDM_DATA16: J17.52, U49.D36
- new net PDM_DATA17: J18.52, U52.D36
- new net PDM_DATA18: J19.52, U55.D36
- new net PDM_DATA19: J20.52, U58.D36
- new net PWM32: J17.32, U49.~D44
- new net PWM33: J17.47, U49.~D45
- new net PWM34: J18.32, U52.~D44
- new net PWM35: J18.47, U52.~D45
- new net PWM36: J19.32, U55.~D44
- new net PWM37: J19.47, U55.~D45
- new net PWM38: J20.32, U58.~D44
- new net PWM39: J20.47, U58.~D45
- new net RTS17: J17.13, U49.D10
- new net RTS18: J18.13, U52.D10
- new net RTS19: J19.13, U55.D10
- new net RTS20: J20.13, U58.D10
- new net RX17: J17.19, U49.~D25
- new net RX18: J18.19, U52.~D25
- new net RX19: J19.19, U55.~D25
- new net RX20: J20.19, U58.~D25
- new net RXI-16: U49.RXI-0, U50.8
- new net RXI-17: U52.RXI-0, U53.8
- new net RXI-18: U55.RXI-0, U56.8
- new net RXI-19: U58.RXI-0, U59.8
- new net SCALED_ADC32: U49.~AD32, U51.5, U51.6
- new net SCALED_ADC33: U49.~AD35, U51.7, U51.8
- new net SCALED_ADC34: U52.~AD32, U54.5, U54.6
- new net SCALED_ADC35: U52.~AD35, U54.7, U54.8
- new net SCALED_ADC36: U55.~AD32, U57.5, U57.6
- new net SCALED_ADC37: U55.~AD35, U57.7, U57.8
- new net SCALED_ADC38: U58.~AD32, U60.5, U60.6
- new net SCALED_ADC39: U58.~AD35, U60.7, U60.8
- new net SCALED_BATT_VIN/17: R148.1, R149.2, U49.~AD31
- new net SCALED_BATT_VIN/18: R157.1, R158.2, U52.~AD31
- new net SCALED_BATT_VIN/19: R166.1, R167.2, U55.~AD31
- new net SCALED_BATT_VIN/20: R175.1, R176.2, U58.~AD31
- new net SCL32: J17.14, U49.~D39
- new net SCL33: J17.55, U49.D8
- new net SCL34: J18.14, U52.~D39
- new net SCL35: J18.55, U52.D8
- new net SCL36: J19.14, U55.~D39
- new net SCL37: J19.55, U55.D8
- new net SCL38: J20.14, U58.~D39
- new net SCL39: J20.55, U58.D8
- new net SDA32: J17.12, U49.D40
- new net SDA33: J17.53, U49.D9
- new net SDA34: J18.12, U52.D40
- new net SDA35: J18.53, U52.D9
- new net SDA36: J19.12, U55.D40
- new net SDA37: J19.53, U55.D9
- new net SDA38: J20.12, U58.D40
- new net SDA39: J20.53, U58.D9
- new net SPI_!CS!16: J9.70, U25.~D23
- new net SPI_!CS!17: J9.49, U25.D41
- new net SPI_!CS!18: J10.70, U28.~D23
- new net SPI_!CS!19: J10.49, U28.D41
- new net SPI_!CS!21: J11.49, U31.D41
- new net SPI_!CS!23: J12.49, U34.D41
- new net SPI_!CS!25: J13.49, U37.D41
- new net SPI_!CS!27: J14.49, U40.D41
- new net SPI_!CS!29: J15.49, U43.D41
- new net SPI_!CS!31: J16.49, U46.D41
- new net SPI_!CS!32: J17.70, U49.~D23
- new net SPI_!CS!33: J17.49, U49.D41
- new net SPI_!CS!34: J18.70, U52.~D23
- new net SPI_!CS!35: J18.49, U52.D41
- new net SPI_!CS!36: J19.70, U55.~D23
- new net SPI_!CS!37: J19.49, U55.D41
- new net SPI_!CS!38: J20.70, U58.~D23
- new net SPI_!CS!39: J20.49, U58.D41
- new net SPI_MISO16: J9.64, U25.~D22, U25.~D6
- new net SPI_MISO17: J9.61, U25.~D43
- new net SPI_MISO18: J10.64, U28.~D22, U28.~D6
- new net SPI_MISO19: J10.61, U28.~D43
- new net SPI_MISO20: J11.64, U31.~D22, U31.~D6
- new net SPI_MISO21: J11.61, U31.~D43
- new net SPI_MISO23: J12.61, U34.~D43
- new net SPI_MISO25: J13.61, U37.~D43
- new net SPI_MISO27: J14.61, U40.~D43
- new net SPI_MISO29: J15.61, U43.~D43
- new net SPI_MISO31: J16.61, U46.~D43
- new net SPI_MISO32: J17.64, U49.~D22, U49.~D6
- new net SPI_MISO33: J17.61, U49.~D43
- new net SPI_MISO34: J18.64, U52.~D22, U52.~D6
- new net SPI_MISO35: J18.61, U52.~D43
- new net SPI_MISO36: J19.64, U55.~D22, U55.~D6
- new net SPI_MISO37: J19.61, U55.~D43
- new net SPI_MISO38: J20.64, U58.~D22, U58.~D6
- new net SPI_MISO39: J20.61, U58.~D43
- new net SPI_MOSI32: J17.59, U49.D38
- new net SPI_MOSI33: J17.62, U49.D7
- new net SPI_MOSI34: J18.59, U52.D38
- new net SPI_MOSI35: J18.62, U52.D7
- new net SPI_MOSI36: J19.59, U55.D38
- new net SPI_MOSI37: J19.62, U55.D7
- new net SPI_MOSI38: J20.59, U58.D38
- new net SPI_MOSI39: J20.62, U58.D7
- new net SPI_SCK32: J17.57, U49.~D42
- new net SPI_SCK33: J17.60, U49.~D5
- new net SPI_SCK34: J18.57, U52.~D42
- new net SPI_SCK35: J18.60, U52.~D5
- new net SPI_SCK36: J19.57, U55.~D42
- new net SPI_SCK37: J19.60, U55.~D5
- new net SPI_SCK38: J20.57, U58.~D42
- new net SPI_SCK39: J20.60, U58.~D5
- new net SWDCK16: J17.21, U49.SWDCK
- new net SWDCK17: J18.21, U52.SWDCK
- new net SWDCK18: J19.21, U55.SWDCK
- new net SWDCK19: J20.21, U58.SWDCK
- new net SWDIO16: J17.23, U49.SWDIO
- new net SWDIO17: J18.23, U52.SWDIO
- new net SWDIO18: J19.23, U55.SWDIO
- new net SWDIO19: J20.23, U58.SWDIO
- new net TX17: J17.17, U49.~D24
- new net TX18: J18.17, U52.~D24
- new net TX19: J19.17, U55.~D24
- new net TX20: J20.17, U58.~D24
- new net TXO-16: U49.TXO-0, U50.9
- new net TXO-17: U52.TXO-0, U53.9
- new net TXO-18: U55.TXO-0, U56.9
- new net TXO-19: U58.TXO-0, U59.9
- new net USB_D+16: J17.3, U50.1
- new net USB_D+17: J18.3, U53.1
- new net USB_D+18: J19.3, U56.1
- new net USB_D+19: J20.3, U59.1
- new net USB_D-16: J17.5, U50.2
- new net USB_D-17: J18.5, U53.2
- new net USB_D-18: J19.5, U56.2
- new net USB_D-19: J20.5, U59.2
- net 3.3V: now also D7.C; no longer J1.2, J1.74
- net 3.3V1: now also D3.C; no longer J2.2, J2.74
- net 3.3V10: now also D22.C; no longer J11.2, J11.74
- net 3.3V11: now also D24.C; no longer J12.2, J12.74
- net 3.3V12: now also D26.C; no longer J13.2, J13.74
- net 3.3V13: now also D28.C; no longer J14.2, J14.74
- net 3.3V14: now also D30.C; no longer J15.2, J15.74
- net 3.3V15: now also D32.C; no longer J16.2, J16.74
- net 3.3V2: now also D5.C; no longer J3.2, J3.74
- net 3.3V3: now also D8.C; no longer J4.2, J4.74
- net 3.3V4: now also D10.C; no longer J5.2, J5.74
- net 3.3V5: now also D12.C; no longer J6.2, J6.74
- net 3.3V6: now also D14.C; no longer J7.2, J7.74
- net 3.3V7: now also D16.C; no longer J8.2, J8.74
- net 3.3V8: now also D18.C; no longer J9.2, J9.74
- net 3.3V9: now also D20.C; no longer J10.2, J10.74
- net CLKOUT: now also J1.58
- net CLKOUT1: now also J2.58
- net CLKOUT10: now also J11.58
- net CLKOUT11: now also J12.58
- net CLKOUT12: now also J13.58
- net CLKOUT13: now also J14.58
- net CLKOUT14: now also J15.58
- net CLKOUT15: now also J16.58
- net CLKOUT2: now also J3.58
- net CLKOUT3: now also J4.58
- net CLKOUT4: now also J5.58
- net CLKOUT5: now also J6.58
- net CLKOUT6: now also J7.58
- net CLKOUT7: now also J8.58
- net CLKOUT8: now also J9.58
- net CLKOUT9: now also J10.58
- net GND: now also J1.GND1, J1.GND2, J1.GND3; no longer J1.GND, J1.GND-SM-B
- net GND1: now also J2.GND1, J2.GND2, J2.GND3; no longer J2.GND, J2.GND-SM-B
- net GND10: now also D21.C, J11.GND1, J11.GND2, J11.GND3; no longer D11.C, J11.GND, J11.GND-SM-B
- net GND11: now also D23.C, J12.GND1, J12.GND2, J12.GND3; no longer D12.C, J12.GND, J12.GND-SM-B
- net GND12: now also D25.C, J13.GND1, J13.GND2, J13.GND3; no longer D13.C, J13.GND, J13.GND-SM-B
- net GND13: now also D27.C, J14.GND1, J14.GND2, J14.GND3; no longer D14.C, J14.GND, J14.GND-SM-B
- net GND14: now also D29.C, J15.GND1, J15.GND2, J15.GND3; no longer D15.C, J15.GND, J15.GND-SM-B
- net GND15: now also D31.C, J16.GND1, J16.GND2, J16.GND3; no longer D16.C, J16.GND, J16.GND-SM-B
- net GND2: now also D4.C, J3.GND1, J3.GND2, J3.GND3; no longer D3.C, J3.GND, J3.GND-SM-B
- net GND3: now also D6.C, J4.GND1, J4.GND2, J4.GND3; no longer D4.C, J4.GND, J4.GND-SM-B
- net GND4: now also D9.C, J5.GND1, J5.GND2, J5.GND3; no longer D5.C, J5.GND, J5.GND-SM-B
- net GND5: now also D11.C, J6.GND1, J6.GND2, J6.GND3; no longer D6.C, J6.GND, J6.GND-SM-B
- net GND6: now also D13.C, J7.GND1, J7.GND2, J7.GND3; no longer D7.C, J7.GND, J7.GND-SM-B
- net GND7: now also D15.C, J8.GND1, J8.GND2, J8.GND3; no longer D8.C, J8.GND, J8.GND-SM-B
- net GND8: now also D17.C, J9.GND1, J9.GND2, J9.GND3; no longer D9.C, J9.GND, J9.GND-SM-B
- net GND9: now also D19.C, J10.GND1, J10.GND2, J10.GND3; no longer D10.C, J10.GND, J10.GND-SM-B
- net N$10: now also D4.A; no longer D3.A
- net N$14: now also D6.A; no longer D4.A
- net N$18: now also D9.A; no longer D5.A
- net N$22: now also D11.A; no longer D6.A
- net N$26: now also D13.A; no longer D7.A
- net N$30: now also D15.A; no longer D8.A
- net N$34: now also D17.A; no longer D9.A
- net N$38: now also D19.A; no longer D10.A
- net N$42: now also D21.A; no longer D11.A
- net N$46: now also D23.A; no longer D12.A
- net N$50: now also D25.A; no longer D13.A
- net N$54: now also D27.A; no longer D14.A
- net N$58: now also D29.A; no longer D15.A
- net N$62: now also D31.A; no longer D16.A
- net SDIO_DATA10: now also J5.68, U13.~D4; no longer J3.66, U7.~D26
- net SDIO_DATA11: now also J6.66, U16.~D26; no longer J3.68, U7.~D4
- net SDIO_DATA12: now also J6.68, U16.~D4; no longer J4.64, U10.~D22, U10.~D6
- net SDIO_DATA13: now also J7.66, U19.~D26; no longer J4.70, U10.~D23
- net SDIO_DATA14: now also J7.68, U19.~D4; no longer J4.66, U10.~D26
- net SDIO_DATA15: now also J8.66, U22.~D26; no longer J4.68, U10.~D4
- net SDIO_DATA16: now also J8.68, U22.~D4; no longer J5.64, U13.~D22, U13.~D6
- net SDIO_DATA17: now also J9.66, U25.~D26; no longer J5.70, U13.~D23
- net SDIO_DATA18: now also J9.68, U25.~D4; no longer J5.66, U13.~D26
- net SDIO_DATA19: now also J10.66, U28.~D26; no longer J5.68, U13.~D4
- net SDIO_DATA20: now also J10.68, U28.~D4; no longer J6.64, U16.~D22, U16.~D6
- net SDIO_DATA21: now also J11.66, U31.~D26; no longer J6.70, U16.~D23
- net SDIO_DATA22: now also J11.68, U31.~D4; no longer J6.66, U16.~D26
- net SDIO_DATA23: now also J12.66, U34.~D26; no longer J6.68, U16.~D4
- net SDIO_DATA24: now also J12.68, U34.~D4; no longer J7.64, U19.~D22, U19.~D6
- net SDIO_DATA25: now also J13.66, U37.~D26; no longer J7.70, U19.~D23
- net SDIO_DATA26: now also J13.68, U37.~D4; no longer J7.66, U19.~D26
- net SDIO_DATA27: now also J14.66, U40.~D26; no longer J7.68, U19.~D4
- net SDIO_DATA28: now also J14.68, U40.~D4; no longer J8.64, U22.~D22, U22.~D6
- net SDIO_DATA29: now also J15.66, U43.~D26; no longer J8.70, U22.~D23
- net SDIO_DATA3: now also J2.66, U3.~D26; no longer J1.70, U1.~D23
- net SDIO_DATA30: now also J15.68, U43.~D4; no longer J8.66, U22.~D26
- net SDIO_DATA31: now also J16.66, U46.~D26; no longer J8.68, U22.~D4
- net SDIO_DATA32: now also J16.68, U46.~D4; no longer J9.64, U25.~D22, U25.~D6
- net SDIO_DATA33: now also J17.66, U49.~D26; no longer J9.70, U25.~D23
- net SDIO_DATA34: now also J17.68, U49.~D4; no longer J9.66, U25.~D26
- net SDIO_DATA35: now also J18.66, U52.~D26; no longer J9.68, U25.~D4
- net SDIO_DATA36: now also J18.68, U52.~D4; no longer J10.64, U28.~D22, U28.~D6
- net SDIO_DATA37: now also J19.66, U55.~D26; no longer J10.70, U28.~D23
- net SDIO_DATA38: now also J19.68, U55.~D4; no longer J10.66, U28.~D26
- net SDIO_DATA39: now also J20.66, U58.~D26; no longer J10.68, U28.~D4
- net SDIO_DATA4: now also J2.68, U3.~D4; no longer J2.64, U3.~D22, U3.~D6
- net SDIO_DATA40: now also J20.68, U58.~D4; no longer J11.64, U31.~D22, U31.~D6
- net SDIO_DATA5: now also J3.66, U7.~D26; no longer J2.70, U3.~D23
- net SDIO_DATA6: now also J3.68, U7.~D4; no longer J2.66, U3.~D26
- net SDIO_DATA7: now also J4.66, U10.~D26; no longer J2.68, U3.~D4
- net SDIO_DATA8: now also J4.68, U10.~D4; no longer J3.64, U7.~D22, U7.~D6
- net SDIO_DATA9: now also J5.66, U13.~D26; no longer J3.70, U7.~D23
- net SPI_!CS!: now also J1.70, U1.~D23; no longer J1.49, U1.D41
- net SPI_!CS!1: now also J1.49, U1.D41; no longer J2.49, U3.D41
- net SPI_!CS!10: now also J6.70, U16.~D23; no longer J11.49, U31.D41
- net SPI_!CS!11: now also J6.49, U16.D41; no longer J12.49, U34.D41
- net SPI_!CS!12: now also J7.70, U19.~D23; no longer J13.49, U37.D41
- net SPI_!CS!13: now also J7.49, U19.D41; no longer J14.49, U40.D41
- net SPI_!CS!14: now also J8.70, U22.~D23; no longer J15.49, U43.D41
- net SPI_!CS!15: now also J8.49, U22.D41; no longer J16.49, U46.D41
- net SPI_!CS!2: now also J2.70, U3.~D23; no longer J3.49, U7.D41
- net SPI_!CS!3: now also J2.49, U3.D41; no longer J4.49, U10.D41
- net SPI_!CS!4: now also J3.70, U7.~D23; no longer J5.49, U13.D41
- net SPI_!CS!5: now also J3.49, U7.D41; no longer J6.49, U16.D41
- net SPI_!CS!6: now also J4.70, U10.~D23; no longer J7.49, U19.D41
- net SPI_!CS!7: now also J4.49, U10.D41; no longer J8.49, U22.D41
- net SPI_!CS!8: now also J5.70, U13.~D23; no longer J9.49, U25.D41
- net SPI_!CS!9: now also J5.49, U13.D41; no longer J10.49, U28.D41
- net SPI_MISO: now also J1.64, U1.~D22, U1.~D6; no longer J1.61, U1.~D43
- net SPI_MISO1: now also J1.61, U1.~D43; no longer J2.61, U3.~D43
- net SPI_MISO10: now also J6.64, U16.~D22, U16.~D6; no longer J11.61, U31.~D43
- net SPI_MISO11: now also J6.61, U16.~D43; no longer J12.61, U34.~D43
- net SPI_MISO12: now also J7.64, U19.~D22, U19.~D6; no longer J13.61, U37.~D43
- net SPI_MISO13: now also J7.61, U19.~D43; no longer J14.61, U40.~D43
- net SPI_MISO14: now also J8.64, U22.~D22, U22.~D6; no longer J15.61, U43.~D43
- net SPI_MISO15: now also J8.61, U22.~D43; no longer J16.61, U46.~D43
- net SPI_MISO2: now also J2.64, U3.~D22, U3.~D6; no longer J3.61, U7.~D43
- net SPI_MISO3: now also J2.61, U3.~D43; no longer J4.61, U10.~D43
- net SPI_MISO4: now also J3.64, U7.~D22, U7.~D6; no longer J5.61, U13.~D43
- net SPI_MISO5: now also J3.61, U7.~D43; no longer J6.61, U16.~D43
- net SPI_MISO6: now also J4.64, U10.~D22, U10.~D6; no longer J7.61, U19.~D43
- net SPI_MISO7: now also J4.61, U10.~D43; no longer J8.61, U22.~D43
- net SPI_MISO8: now also J5.64, U13.~D22, U13.~D6; no longer J9.61, U25.~D43
- net SPI_MISO9: now also J5.61, U13.~D43; no longer J10.61, U28.~D43
- net SPI_MOSI: now also J1.62, U1.D7; no longer J1.59, U1.D38
- net SPI_MOSI1: now also J1.59, U1.D38; no longer J1.62, U1.D7
- net SPI_SCK: now also J1.60, U1.~D5; no longer J1.57, U1.~D42
- net SPI_SCK1: now also J1.57, U1.~D42; no longer J1.60, U1.~D5
Routing:
- net GPIO136: track 0.00 -> 41.7 mm, vias 0 -> 2
- net GPIO128: track 0.00 -> 41.7 mm, vias 0 -> 2
- net GPIO152: track 0.00 -> 41.7 mm, vias 0 -> 2
- net GPIO144: track 0.00 -> 41.7 mm, vias 0 -> 2
- net CLKOUT19: track 0.00 -> 33.6 mm, vias 0 -> 3
- net CLKOUT18: track 0.00 -> 33.6 mm, vias 0 -> 3
- net CLKOUT17: track 0.00 -> 33.6 mm, vias 0 -> 3
- net CLKOUT16: track 0.00 -> 33.6 mm, vias 0 -> 3
- net SPI_MISO39: track 0.00 -> 32.5 mm
- net SPI_MISO37: track 0.00 -> 32.5 mm
- net SPI_MISO29: track 0.00 -> 32.5 mm
- net SPI_MISO27: track 0.00 -> 32.5 mm
- net SPI_MISO23: track 0.00 -> 32.5 mm
- net SPI_MISO21: track 0.00 -> 32.5 mm
- net SPI_MISO19: track 0.00 -> 32.5 mm
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- added copper zone on layer 15, net 3.3V16
- added copper zone on layer 15, net 3.3V17
- added copper zone on layer 15, net 3.3V18
- added copper zone on layer 15, net 3.3V19
- added copper zone on layer 1, net GND16
- added copper zone on layer 15, net GND16
- added copper zone on layer 16, net GND16
- added copper zone on layer 2, net GND16
- added copper zone on layer 1, net GND17
- added copper zone on layer 15, net GND17
- added copper zone on layer 16, net GND17
- added copper zone on layer 2, net GND17
- added copper zone on layer 1, net GND18
- added copper zone on layer 15, net GND18
- added copper zone on layer 16, net GND18
- added copper zone on layer 2, net GND18
- added copper zone on layer 1, net GND19
- added copper zone on layer 15, net GND19
- added copper zone on layer 16, net GND19
- added copper zone on layer 2, net GND19
Other:
- board size 199.6 x 83.1 mm -> 244.6 x 83.1 mm
- board text added: "Do not remove"
- board text added: "v12"
- board text removed: "v11"
