File: Hardware/MicroMod-Artemis-ProcessorBoard.sch (EAGLE design)
At the start: 33 parts, among them J1 MICROMOD-2222, U1 ARTEMIS_MODULESMD, U2 TSV524, U6 CH340E_MSOP10, Y1 32.768kHz

Commit message: Add missing net to Xtal
Connections:
- removed net N$4: U1.XI
- net N$5: now also U1.XI
Other:
- note added: "30uA (typ) per channel"
- note added: "Connect D24 to SDIO_CLK Move TX1 from D24 to somewhere else consider 1,7,10,15,19,28 for CE0/!CS!"
Changed lines of the file:
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@@
 <?xml version="1.0" encoding="utf-8"?>
 <!DOCTYPE eagle SYSTEM "eagle.dtd">
-<eagle version="9.6.0">
+<eagle version="9.6.2">
 <drawing>
 <settings>
@@
 <text x="71.374" y="119.126" size="2.54" layer="97" font="vector" align="center">Bootloader Reset Circuit</text>
 <text x="213.614" y="266.446" size="2.54" layer="97" font="vector" align="center">MicroMod Connector</text>
-<text x="343.154" y="248.666" size="2.54" layer="97" font="vector" align="center">3.3V to 2V Scaling</text>
+<text x="342.9" y="246.38" size="2.54" layer="97" font="vector" align="center">3.3V to 2V Scaling</text>
 <text x="421.64" y="7.62" size="2.54" layer="94">v1.2</text>
 <text x="348.742" y="11.176" size="2.54" layer="94">N. Seidle</text>
@@
 <text x="176.276" y="257.302" size="1.778" layer="97">0.65uA Leakage
 0.3V drop at 10mA</text>
+<text x="340.36" y="99.06" size="1.27" layer="91">Connect D24 to SDIO_CLK
+Move TX1 from D24 to somewhere else
+consider 1,7,10,15,19,28 for CE0/!CS!</text>
+<text x="342.9" y="243.84" size="1.27" layer="97" align="center">30uA (typ) per channel</text>
 </plain>
 <instances>
@@
 </segment>
 </net>
-<net name="N$8" class="0">
-<segment>
-<wire x1="42.4942" y1="210.82" x2="30.48" y2="210.82" width="0.1524" layer="91"/>
-<wire x1="30.48" y1="210.82" x2="30.48" y2="213.1303625" width="0.1524" layer="91"/>
-</segment>
-</net>
 <net name="N$2" class="0">
 <segment>
@@
 </segment>
 </net>
-<net name="N$4" class="0">
-<segment>
-<pinref part="U1" gate="U1" pin="XI"/>
-<wire x1="43.18" y1="210.82" x2="42.8498" y2="210.82" width="0.1524" layer="91"/>
-</segment>
-</net>
 <net name="N$5" class="0">
 <segment>
 <pinref part="C13" gate="G$1" pin="2"/>
 <wire x1="27.94" y1="213.36" x2="25.4" y2="213.36" width="0.1524" layer="91"/>
-<junction x="27.94" y="213.36"/>
 <pinref part="Y1" gate="G$1" pin="1"/>
 <wire x1="27.94" y1="210.82" x2="27.94" y2="213.36" width="0.1524" layer="91"/>
-<wire x1="30.0482" y1="213.36" x2="27.94" y2="213.36" width="0.1524" layer="91"/>
-</segment>
-</net>
-<net name="N$6" class="0">
-<segment>
-<wire x1="30.48" y1="213.36" x2="30.4038" y2="213.36" width="0.1524" layer="91"/>
-</segment>
-</net>
+<pinref part="U1" gate="U1" pin="XI"/>
+<wire x1="43.18" y1="210.82" x2="30.48" y2="210.82" width="0.1524" layer="91"/>
+<wire x1="30.48" y1="210.82" x2="30.48" y2="213.36" width="0.1524" layer="91"/>
+<wire x1="30.48" y1="213.36" x2="27.94" y2="213.36" width="0.1524" layer="91"/>
+<junction x="27.94" y="213.36"/>
+</segment>
+</net>

Commit message: Fix SDA1/SCL1, CS1, and VIN/3 incorrect pin locations.
Changed lines of the file:
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@@
 <?xml version="1.0" encoding="utf-8"?>
 <!DOCTYPE eagle SYSTEM "eagle.dtd">
-<eagle version="9.6.2">
+<eagle version="9.6.0">
 <drawing>
 <settings>
@@
 <net name="BATT_VIN/3" class="0">
 <segment>
-<wire x1="190.5" y1="167.64" x2="187.96" y2="167.64" width="0.1524" layer="91"/>
-<label x="187.96" y="167.64" size="1.27" layer="95" rot="R180" xref="yes"/>
-<pinref part="J1" gate="J1" pin="BATT_VIN/3"/>
-</segment>
-<segment>
 <pinref part="R2" gate="G$1" pin="2"/>
 <wire x1="353.06" y1="187.96" x2="353.06" y2="190.5" width="0.1524" layer="91"/>
@@
 <label x="350.52" y="190.5" size="1.27" layer="95" rot="R180" xref="yes"/>
 </segment>
+<segment>
+<pinref part="J1" gate="J1" pin="BATT_VIN/3"/>
+<wire x1="190.5" y1="167.64" x2="187.96" y2="167.64" width="0.1524" layer="91"/>
+<label x="187.96" y="167.64" size="1.27" layer="95" rot="R180" xref="yes"/>
+</segment>
 </net>
 <net name="ADC0" class="0">
@@
 </segment>
 <segment>
+<pinref part="J1" gate="J1" pin="I2C_SCL1"/>
 <wire x1="190.5" y1="175.26" x2="187.96" y2="175.26" width="0.1524" layer="91"/>
 <label x="187.96" y="175.26" size="1.27" layer="95" rot="R180" xref="yes"/>
-<pinref part="J1" gate="J1" pin="I2C_SCL1"/>
 </segment>
 </net>
@@
 </segment>
 <segment>
+<pinref part="J1" gate="J1" pin="I2C_SDA1"/>
 <wire x1="190.5" y1="172.72" x2="187.96" y2="172.72" width="0.1524" layer="91"/>
 <label x="187.96" y="172.72" size="1.27" layer="95" rot="R180" xref="yes"/>
-<pinref part="J1" gate="J1" pin="I2C_SDA1"/>
 </segment>
 </net>
@@
 </segment>
 <segment>
+<pinref part="J1" gate="J1" pin="SPI_!CS!1"/>
 <wire x1="236.22" y1="223.52" x2="238.76" y2="223.52" width="0.1524" layer="91"/>
 <label x="238.76" y="223.52" size="1.27" layer="95" xref="yes"/>
-<pinref part="J1" gate="J1" pin="SPI_!CS!1"/>
-</segment>
-</net>
+</segment>
+</net>

Commit message: Roll version to v1.4
Other:
- note added: "v1.4"
- note removed: "v1.2"
Changed lines of the file:
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@@
 <text x="213.614" y="266.446" size="2.54" layer="97" font="vector" align="center">MicroMod Connector</text>
 <text x="342.9" y="246.38" size="2.54" layer="97" font="vector" align="center">3.3V to 2V Scaling</text>
-<text x="421.64" y="7.62" size="2.54" layer="94">v1.2</text>
+<text x="421.64" y="7.62" size="2.54" layer="94">v1.4</text>
 <text x="348.742" y="11.176" size="2.54" layer="94">N. Seidle</text>
 <text x="76.454" y="256.286" size="2.54" layer="97" font="vector" align="center">Artemis</text>

Commit message: Connect SPI pins to support Quad SPI. Move TX1 to AD12
Connections:
- net SDIO_DATA1 renamed QSPI1
- net SDIO_DATA2 renamed QSPI2
- net SPI_!CS! renamed SPI_!CS!/QSPI3
- removed net ADC_D-: J1.G9/ADC_D-/CAM_HSYNC, U1.~AD12(PDMCLK/TX1)
- removed net SPI_MISO: J1.SPI_MISO/SDIO_DATA0, U1.(PDMCLK/SWO)~D22, U1.(SDA0/MISO0/I2SDAT)~D6
- removed net SPI_MOSI: J1.SPI_MOSI/SDIO_CMD, U1.(MOSI0/CLKOUT)~D7
- removed net SPI_SCK: J1.SPI_SCK/SDIO_CLK, U1.(SCL0/SCK0)~D5
- removed net TX1: J1.TX1, U1.(TX1/32KHZ/SWO)~D24
- new net SPI_MISO/QSPI0: J1.SPI_SDI/SDIO_DATA0, U1.(PDMCLK/SWO)~D22, U1.(SDA0/SDI0/I2SDAT)~D6
- new net SPI_MOSI/QSPI_!CS!: J1.SPI_SDO/SDIO_CMD, U1.(SDO0/CLKOUT)~D7
- new net SPI_SCK/QSPI_CLK: J1.SPI_SCK/SDIO_CLK, U1.(SCL0/SCK0)~D5, U1.(TX1/32KHZ/SWO)~D24
- new net TX1/ADC_D-: J1.G9/ADC_D-/CAM_HSYNC, J1.TX1, U1.~AD12(PDMCLK/TX1)
- net BOOT: now also U1.~BOOT(SDO5/RX1/32KHZ); no longer U1.~BOOT(MOSI5/RX1/32KHZ)
- net D0: now also U1.(SLSDO/SLSDA)D1; no longer U1.(SLMOSI/SLSDA)D1
- net D1: now also U1.(SLSDI)D2; no longer U1.(SLMISO)D2
- net GPIO4: now also U1.(SDO2/I2SWCLK)~D28; no longer U1.(MOSI2/I2SWCLK)~D28
- net PWM0: now also U1.(SDO4)~D44; no longer U1.(MOSI4)~D44
- net RTS1: now also U1.(SDO1/TX1/PDMCLK)D10; no longer U1.(MOSI1/TX1/PDMCLK)D10
- net RX1: now also U1.(SDA2/SDI2/RX1)~D25; no longer U1.(SDA2/MISO2/RX1)~D25
- net RXI-0: now also U1.~D49(RX0/SDA5/SDI5); no longer U1.~D49(RX0/SDA5/MISO5)
- net SDA: now also U1.(SDA4/SDI4/RX1)D40; no longer U1.(SDA4/MISO4/RX1)D40
- net SDA1: now also U1.(SDA1/SDI1/RX1/SCCIO)D9; no longer U1.(SDA1/MISO1/RX1/SCCIO)D9
- net SPI_MISO1: now also J1.SPI_SDI1, U1.(SDA3/SDI3/RX1)~D43; no longer J1.SPI_MISO1, U1.(SDA3/MISO3/RX1)~D43
- net SPI_MOSI1: now also J1.SPI_SDO1, U1.(SDO3/RX1)D38; no longer J1.SPI_MOSI1, U1.(MOSI3/RX1)D38
Other:
- note removed: "Connect D24 to SDIO_CLK Move TX1 from D24 to somewhere else consider 1,7,10,15,19,28 for CE0/!CS!"

Commit message: Adding additional decoupling, change version to v16.
Parts:
- added C2: 0.22uF, SparkFun-Capacitors:0.22UF-0402T-10V-10%
- added C3: 1.0uF, SparkFun-Capacitors:1.0UF-0402T-16V-10%
- added C4: 10uF, SparkFun-Capacitors:10UF-0603-6.3V-20%
- R15: value 220KOHM-0402T-1/16W-1% -> 220K
Connections:
- net SPI_SCK/QSPI_CLK renamed SPI_SCK/QSPI_SCK
- removed net CLKOUT: J1.AUD_MCLK, J1.AUD_OUT/CAM_MCLK, U1.(SLSCK/SLSCL/CLKOUT)D0
- new net CAM_MCLK: J1.AUD_MCLK, J1.AUD_OUT/CAM_MCLK, U1.(CMPIN1/SCCIO)~D18
- net 3.3V: now also C2.1, C3.1, C4.1
- net D0: now also U1.(SLSCK/SLSCL/CLKOUT)D0; no longer U1.(SLSDO/SLSDA)D1
- net D1: now also U1.(SLSDO/SLSDA)D1; no longer U1.(SLSDI)D2
- net GND: now also C2.2, C3.2, C4.2
- net I2C_!INT!: now also U1.(SLSDI)D2; no longer U1.(CMPIN1/SCCIO)~D18
Other:
- note added: "v1.6"
- note removed: "v1.4"
Changed lines of the file:
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@@
 <part name="C20" library="SparkFun-Capacitors" deviceset="0.1UF" device="-0402T-16V-10%" value="0.1uF"/>
 <part name="GND41" library="SparkFun-PowerSymbols" deviceset="GND" device=""/>
-<part name="R15" library="SparkFun-Resistors" deviceset="220KOHM" device="-0402T-1/16W-1%" value="220KOHM-0402T-1/16W-1%"/>
+<part name="R15" library="SparkFun-Resistors" deviceset="220KOHM" device="-0402T-1/16W-1%" value="220K"/>
 <part name="C21" library="SparkFun-Capacitors" deviceset="0.1UF" device="-0402T-16V-10%" value="0.1uF"/>
 <part name="C28" library="SparkFun-Capacitors" deviceset="1.0NF/1000PF" device="-0402_TIGHT-50V-10%" value="1.0nF"/>
@@
 <part name="LOGO2" library="SparkFun-Aesthetics" deviceset="SFE_LOGO_FLAME" device=".1_INCH"/>
 <part name="J1" library="SparkFun-MicroMod" deviceset="MICROMOD" device="-2222"/>
+<part name="C2" library="SparkFun-Capacitors" deviceset="0.22UF" device="-0402T-10V-10%" value="0.22uF"/>
+<part name="C3" library="SparkFun-Capacitors" deviceset="1.0UF" device="-0402T-16V-10%" value="1.0uF"/>
+<part name="C4" library="SparkFun-Capacitors" deviceset="10UF" device="-0603-6.3V-20%" value="10uF"/>
+<part name="SUPPLY5" library="SparkFun-PowerSymbols" deviceset="3.3V" device=""/>
+<part name="SUPPLY6" library="SparkFun-PowerSymbols" deviceset="3.3V" device=""/>
+<part name="SUPPLY7" library="SparkFun-PowerSymbols" deviceset="3.3V" device=""/>
+<part name="GND9" library="SparkFun-PowerSymbols" deviceset="GND" device=""/>
+<part name="GND10" library="SparkFun-PowerSymbols" deviceset="GND" device=""/>
+<part name="GND11" library="SparkFun-PowerSymbols" deviceset="GND" device=""/>
 </parts>
 <sheets>
@@
 <text x="213.614" y="266.446" size="2.54" layer="94" font="vector" align="center">MicroMod Connector</text>
 <text x="342.9" y="246.38" size="2.54" layer="94" font="vector" align="center">3.3V to 2V Scaling</text>
-<text x="421.64" y="7.62" size="2.54" layer="94">v1.4</text>
+<text x="421.64" y="7.62" size="2.54" layer="94">v1.6</text>
 <text x="348.742" y="11.176" size="2.54" layer="94">N. Seidle</text>
 <text x="76.454" y="256.286" size="2.54" layer="94" font="vector" align="center">Artemis</text>
@@
 <text x="176.276" y="257.302" size="1.778" layer="97">0.65uA Leakage
 0.3V drop at 10mA</text>
-<text x="342.9" y="243.84" size="1.27" layer="94" align="center">30uA (typ) per channel</text>
+<text x="342.9" y="243.84" size="1.27" layer="97" align="center">30uA (typ) per channel</text>
 </plain>
 <instances>
@@
 <instance part="R15" gate="G$1" x="63.5" y="93.98" smashed="yes" rot="MR90">
 <attribute name="NAME" x="65.024" y="93.98" size="1.778" layer="95" font="vector" rot="MR90" align="bottom-center"/>
+<attribute name="VALUE" x="61.976" y="93.98" size="1.778" layer="96" font="vector" rot="MR90" align="top-center"/>
 </instance>
 <instance part="C21" gate="G$1" x="58.42" y="101.6" smashed="yes" rot="R90">
@@
 <attribute name="NAME" x="193.04" y="251.968" size="1.778" layer="95"/>
 <attribute name="VALUE" x="193.04" y="149.86" size="1.778" layer="96"/>
+</instance>
+<instance part="C2" gate="G$1" x="30.48" y="30.48" smashed="yes">
+<attribute name="NAME" x="32.004" y="33.401" size="1.778" layer="95" font="vector"/>
+<attribute name="VALUE" x="32.004" y="28.321" size="1.778" layer="96" font="vector"/>
+</instance>
+<instance part="C3" gate="G$1" x="20.32" y="30.48" smashed="yes">
+<attribute name="NAME" x="21.844" y="33.401" size="1.778" layer="95" font="vector"/>
+<attribute name="VALUE" x="21.844" y="28.321" size="1.778" layer="96" font="vector"/>
+</instance>
+<instance part="C4" gate="G$1" x="10.16" y="30.48" smashed="yes">
+<attribute name="NAME" x="11.684" y="33.401" size="1.778" layer="95" font="vector"/>
+<attribute name="VALUE" x="11.684" y="28.321" size="1.778" layer="96" font="vector"/>
+</instance>
+<instance part="SUPPLY5" gate="G$1" x="30.48" y="38.1" smashed="yes">
+<attribute name="VALUE" x="30.48" y="40.894" size="1.778" layer="96" align="bottom-center"/>
+</instance>
+<instance part="SUPPLY6" gate="G$1" x="20.32" y="38.1" smashed="yes">
+<attribute name="VALUE" x="20.32" y="40.894" size="1.778" layer="96" align="bottom-center"/>
+</instance>
+<instance part="SUPPLY7" gate="G$1" x="10.16" y="38.1" smashed="yes">
+<attribute name="VALUE" x="10.16" y="40.894" size="1.778" layer="96" align="bottom-center"/>
+</instance>
+<instance part="GND9" gate="1" x="30.48" y="22.86" smashed="yes">
+<attribute name="VALUE" x="30.48" y="22.606" size="1.778" layer="96" align="top-center"/>
+</instance>
+<instance part="GND10" gate="1" x="20.32" y="22.86" smashed="yes">
+<attribute name="VALUE" x="20.32" y="22.606" size="1.778" layer="96" align="top-center"/>
+</instance>
+<instance part="GND11" gate="1" x="10.16" y="22.86" smashed="yes">
+<attribute name="VALUE" x="10.16" y="22.606" size="1.778" layer="96" align="top-center"/>
 </instance>
 </instances>
@@
 <pinref part="J1" gate="J1" pin="RTC_3V"/>
 </segment>
+<segment>
+<pinref part="C2" gate="G$1" pin="1"/>
+<pinref part="SUPPLY5" gate="G$1" pin="3.3V"/>
+<wire x1="30.48" y1="38.1" x2="30.48" y2="35.56" width="0.1524" layer="91"/>
+</segment>
+<segment>
+<pinref part="C3" gate="G$1" pin="1"/>
+<pinref part="SUPPLY6" gate="G$1" pin="3.3V"/>
+<wire x1="20.32" y1="38.1" x2="20.32" y2="35.56" width="0.1524" layer="91"/>
+</segment>
+<segment>
+<pinref part="C4" gate="G$1" pin="1"/>
+<pinref part="SUPPLY7" gate="G$1" pin="3.3V"/>
+<wire x1="10.16" y1="38.1" x2="10.16" y2="35.56" width="0.1524" layer="91"/>
+</segment>
 </net>
 <net name="GND" class="0">
@@
 <pinref part="GND8" gate="1" pin="GND"/>
 <wire x1="327.66" y1="162.56" x2="327.66" y2="165.1" width="0.1524" layer="91"/>
+</segment>
+<segment>
+<pinref part="C2" gate="G$1" pin="2"/>
+<pinref part="GND9" gate="1" pin="GND"/>
+<wire x1="30.48" y1="27.94" x2="30.48" y2="25.4" width="0.1524" layer="91"/>
+</segment>
+<segment>
+<pinref part="C3" gate="G$1" pin="2"/>
+<pinref part="GND10" gate="1" pin="GND"/>
+<wire x1="20.32" y1="27.94" x2="20.32" y2="25.4" width="0.1524" layer="91"/>
+</segment>
+<segment>
+<pinref part="C4" gate="G$1" pin="2"/>
+<pinref part="GND11" gate="1" pin="GND"/>
+<wire x1="10.16" y1="27.94" x2="10.16" y2="25.4" width="0.1524" layer="91"/>
 </segment>
 </net>
@@
 </segment>
 </net>
-<net name="SPI_SCK/QSPI_CLK" class="0">
+<net name="SPI_SCK/QSPI_SCK" class="0">
 <segment>
 <pinref part="U1" gate="U1" pin="(TX1/32KHZ/SWO)~D24"/>
@@
 </segment>
 <segment>
-<pinref part="U1" gate="U1" pin="(CMPIN1/SCCIO)~D18"/>
-<wire x1="111.76" y1="210.82" x2="114.3" y2="210.82" width="0.1524" layer="91"/>
-<label x="114.3" y="210.82" size="1.27" layer="95" xref="yes"/>
+<pinref part="U1" gate="U1" pin="(SLSDI)D2"/>
+<wire x1="111.76" y1="241.3" x2="114.3" y2="241.3" width="0.1524" layer="91"/>
+<label x="114.3" y="241.3" size="1.27" layer="95" xref="yes"/>
 </segment>
 </net>
@@
 </segment>
 <segment>
+<pinref part="U1" gate="U1" pin="(SLSCK/SLSCL/CLKOUT)D0"/>
+<wire x1="111.76" y1="246.38" x2="114.3" y2="246.38" width="0.1524" layer="91"/>
+<label x="114.3" y="246.38" size="1.27" layer="95" xref="yes"/>
+</segment>
+</net>
+<net name="D1" class="0">
+<segment>
+<wire x1="236.22" y1="205.74" x2="238.76" y2="205.74" width="0.1524" layer="91"/>
+<label x="238.76" y="205.74" size="1.27" layer="95" xref="yes"/>
+<pinref part="J1" gate="J1" pin="D1/CAM_TRIG"/>
+</segment>
+<segment>
 <pinref part="U1" gate="U1" pin="(SLSDO/SLSDA)D1"/>
 <wire x1="111.76" y1="243.84" x2="114.3" y2="243.84" width="0.1524" layer="91"/>
 <label x="114.3" y="243.84" size="1.27" layer="95" xref="yes"/>
-</segment>
-</net>
-<net name="D1" class="0">
-<segment>
-<wire x1="236.22" y1="205.74" x2="238.76" y2="205.74" width="0.1524" layer="91"/>
-<label x="238.76" y="205.74" size="1.27" layer="95" xref="yes"/>
-<pinref part="J1" gate="J1" pin="D1/CAM_TRIG"/>
-</segment>
-<segment>
-<pinref part="U1" gate="U1" pin="(SLSDI)D2"/>
-<wire x1="111.76" y1="241.3" x2="114.3" y2="241.3" width="0.1524" layer="91"/>
-<label x="114.3" y="241.3" size="1.27" layer="95" xref="yes"/>
 </segment>
 </net>
@@
 <wire x1="236.22" y1="223.52" x2="238.76" y2="223.52" width="0.1524" layer="91"/>
 <label x="238.76" y="223.52" size="1.27" layer="95" xref="yes"/>
-</segment>
-</net>
-<net name="CLKOUT" class="0">
-<segment>
-<pinref part="U1" gate="U1" pin="(SLSCK/SLSCL/CLKOUT)D0"/>
-<wire x1="111.76" y1="246.38" x2="114.3" y2="246.38" width="0.1524" layer="91"/>
-<label x="114.3" y="246.38" size="1.27" layer="95" xref="yes"/>
-</segment>
-<segment>
-<wire x1="190.5" y1="195.58" x2="187.96" y2="195.58" width="0.1524" layer="91"/>
-<label x="185.42" y="195.58" size="1.27" layer="95" rot="R180" xref="yes"/>
-<wire x1="187.96" y1="195.58" x2="185.42" y2="195.58" width="0.1524" layer="91"/>
-<wire x1="190.5" y1="198.12" x2="187.96" y2="198.12" width="0.1524" layer="91" style="longdash"/>
-<wire x1="187.96" y1="198.12" x2="187.96" y2="195.58" width="0.1524" layer="91" style="longdash"/>
-<junction x="187.96" y="195.58"/>
-<pinref part="J1" gate="J1" pin="AUD_MCLK"/>
-<pinref part="J1" gate="J1" pin="AUD_OUT/CAM_MCLK"/>
 </segment>
 </net>
@@
 </segment>
 </net>
+<net name="CAM_MCLK" class="0">
+<segment>
+<pinref part="U1" gate="U1" pin="(CMPIN1/SCCIO)~D18"/>
+<wire x1="111.76" y1="210.82" x2="114.3" y2="210.82" width="0.1524" layer="91"/>
+<label x="114.3" y="210.82" size="1.27" layer="95" xref="yes"/>
+</segment>
+<segment>
+<wire x1="190.5" y1="195.58" x2="187.96" y2="195.58" width="0.1524" layer="91"/>
+<label x="185.42" y="195.58" size="1.27" layer="95" rot="R180" xref="yes"/>
+<wire x1="187.96" y1="195.58" x2="185.42" y2="195.58" width="0.1524" layer="91"/>
+<wire x1="190.5" y1="198.12" x2="187.96" y2="198.12" width="0.1524" layer="91" style="longdash"/>
+<wire x1="187.96" y1="198.12" x2="187.96" y2="195.58" width="0.1524" layer="91" style="longdash"/>
+<junction x="187.96" y="195.58"/>
+<pinref part="J1" gate="J1" pin="AUD_MCLK"/>
+<pinref part="J1" gate="J1" pin="AUD_OUT/CAM_MCLK"/>
+</segment>
+</net>

Commit message: Update SPI port 0/1 net names.
Connections:
- removed net SPI_!CS!/QSPI3: J1.SPI_!CS!/SDIO_DATA3, U1.(I2SWCLK/CMPOUT)~D23
- removed net SPI_!CS!1: J1.SPI_!CS!1, U1.(BLEIF_IRQ/SWO/I2SWCLK)D41
- removed net SPI_MISO/QSPI0: J1.SPI_SDI/SDIO_DATA0, U1.(PDMCLK/SWO)~D22, U1.(SDA0/SDI0/I2SDAT)~D6
- removed net SPI_MISO1: J1.SPI_SDI1, U1.(SDA3/SDI3/RX1)~D43
- removed net SPI_MOSI/QSPI_!CS!: J1.SPI_SDO/SDIO_CMD, U1.(SDO0/CLKOUT)~D7
- removed net SPI_MOSI1: J1.SPI_SDO1, U1.(SDO3/RX1)D38
- removed net SPI_SCK/QSPI_SCK: J1.SPI_SCK/SDIO_CLK, U1.(SCL0/SCK0)~D5, U1.(TX1/32KHZ/SWO)~D24
- removed net SPI_SCK1: J1.SPI_SCK1, U1.(SCL3/SCK3/TX1)~D42
- new net SPI_!CS!: J1.SPI_!CS!, U1.(BLEIF_IRQ/SWO/I2SWCLK)D41
- new net SPI_!CS1!/QSPI3: J1.SPI_!CS1!/SDIO_DATA3, U1.(I2SWCLK/CMPOUT)~D23
- new net SPI_CIPO: J1.SPI_SDI, U1.(SDA3/SDI3/RX1)~D43
- new net SPI_CIPO1/QSPI0: J1.SPI_SDI1/SDIO_DATA0, U1.(PDMCLK/SWO)~D22, U1.(SDA0/SDI0/I2SDAT)~D6
- new net SPI_COPI: J1.SPI_SDO, U1.(SDO3/RX1)D38
- new net SPI_COPI1/QSPI_!CS!: J1.SPI_SDO1/SDIO_CMD, U1.(SDO0/CLKOUT)~D7
- new net SPI_SCK: J1.SPI_SCK, U1.(SCL3/SCK3/TX1)~D42
- new net SPI_SCK1/QSPI_SCK: J1.SPI_SCK1/SDIO_CLK, U1.(SCL0/SCK0)~D5, U1.(TX1/32KHZ/SWO)~D24
Changed lines of the file:
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@@
 </segment>
 </net>
-<net name="SPI_SCK1" class="0">
+<net name="SPI_SCK" class="0">
 <segment>
 <wire x1="236.22" y1="231.14" x2="238.76" y2="231.14" width="0.1524" layer="91"/>
 <label x="238.76" y="231.14" size="1.27" layer="95" rot="MR180" xref="yes"/>
-<pinref part="J1" gate="J1" pin="SPI_SCK1"/>
+<pinref part="J1" gate="J1" pin="SPI_SCK"/>
 </segment>
 <segment>
@@
 </segment>
 </net>
-<net name="SPI_MOSI1" class="0">
+<net name="SPI_COPI" class="0">
 <segment>
 <wire x1="236.22" y1="228.6" x2="238.76" y2="228.6" width="0.1524" layer="91"/>
 <label x="238.76" y="228.6" size="1.27" layer="95" rot="MR180" xref="yes"/>
-<pinref part="J1" gate="J1" pin="SPI_SDO1"/>
+<pinref part="J1" gate="J1" pin="SPI_SDO"/>
 </segment>
 <segment>
@@
 </segment>
 </net>
-<net name="SPI_SCK/QSPI_SCK" class="0">
+<net name="SPI_SCK1/QSPI_SCK" class="0">
 <segment>
 <pinref part="U1" gate="U1" pin="(TX1/32KHZ/SWO)~D24"/>
@@
 <wire x1="236.22" y1="248.92" x2="238.76" y2="248.92" width="0.1524" layer="91"/>
 <label x="238.76" y="248.92" size="1.27" layer="95" xref="yes"/>
-<pinref part="J1" gate="J1" pin="SPI_SCK/SDIO_CLK"/>
+<pinref part="J1" gate="J1" pin="SPI_SCK1/SDIO_CLK"/>
 </segment>
 </net>
@@
 </segment>
 </net>
-<net name="SPI_MISO/QSPI0" class="0">
+<net name="SPI_CIPO1/QSPI0" class="0">
 <segment>
 <wire x1="236.22" y1="243.84" x2="238.76" y2="243.84" width="0.1524" layer="91"/>
 <label x="238.76" y="243.84" size="1.27" layer="95" xref="yes"/>
-<pinref part="J1" gate="J1" pin="SPI_SDI/SDIO_DATA0"/>
+<pinref part="J1" gate="J1" pin="SPI_SDI1/SDIO_DATA0"/>
 </segment>
 <segment>
@@
 </segment>
 </net>
-<net name="SPI_MOSI/QSPI_!CS!" class="0">
+<net name="SPI_COPI1/QSPI_!CS!" class="0">
 <segment>
 <pinref part="U1" gate="U1" pin="(SDO0/CLKOUT)~D7"/>
@@
 <wire x1="236.22" y1="246.38" x2="238.76" y2="246.38" width="0.1524" layer="91"/>
 <label x="238.76" y="246.38" size="1.27" layer="95" xref="yes"/>
-<pinref part="J1" gate="J1" pin="SPI_SDO/SDIO_CMD"/>
-</segment>
-</net>
-<net name="SPI_!CS!/QSPI3" class="0">
+<pinref part="J1" gate="J1" pin="SPI_SDO1/SDIO_CMD"/>
+</segment>
+</net>
+<net name="SPI_!CS1!/QSPI3" class="0">
 <segment>
 <wire x1="236.22" y1="236.22" x2="238.76" y2="236.22" width="0.1524" layer="91"/>
 <label x="238.76" y="236.22" size="1.27" layer="95" xref="yes"/>
-<pinref part="J1" gate="J1" pin="SPI_!CS!/SDIO_DATA3"/>
+<pinref part="J1" gate="J1" pin="SPI_!CS1!/SDIO_DATA3"/>
 </segment>
 <segment>
@@
 </segment>
 </net>
-<net name="SPI_MISO1" class="0">
+<net name="SPI_CIPO" class="0">
 <segment>
 <pinref part="U1" gate="U1" pin="(SDA3/SDI3/RX1)~D43"/>
@@
 <wire x1="236.22" y1="226.06" x2="238.76" y2="226.06" width="0.1524" layer="91"/>
 <label x="238.76" y="226.06" size="1.27" layer="95" rot="MR180" xref="yes"/>
-<pinref part="J1" gate="J1" pin="SPI_SDI1"/>
+<pinref part="J1" gate="J1" pin="SPI_SDI"/>
 </segment>
 </net>
@@
 </segment>
 </net>
-<net name="SPI_!CS!1" class="0">
+<net name="SPI_!CS!" class="0">
 <segment>
 <pinref part="U1" gate="U1" pin="(BLEIF_IRQ/SWO/I2SWCLK)D41"/>
@@
 </segment>
 <segment>
-<pinref part="J1" gate="J1" pin="SPI_!CS!1"/>
+<pinref part="J1" gate="J1" pin="SPI_!CS!"/>
 <wire x1="236.22" y1="223.52" x2="238.76" y2="223.52" width="0.1524" layer="91"/>
 <label x="238.76" y="223.52" size="1.27" layer="95" xref="yes"/>
